File: CellMan.kicad_pcb (KiCad board)
At the start: 2 copper layers, 100 x 45 mm, 58 parts, among them J1 Conn_01x04_Female, J2 Conn_01x04_Male, J3 Conn_01x04_Male, J4 Conn_01x06_Female, J5 Conn_01x02_Female, J6 Conn_01x02_Female, J7 Conn_01x03_Male, Q1 BSS138W, SW1 SW_DIP_x06, SW2 SW_DIP_x04, U1 ADC128D818, U2 MCP9808, U3 MCP6004

Commit message: idk, theres ovals now
Parts:
- removed C3, C4: C, Capacitor_SMD:C_0805_2012Metric_Pad1.15x1.40mm_HandSolder
- removed G***: LOGO, Lafayette_Electric_Car_Footprints:paw_solder_mask
- removed G***: LOGO, Lafayette_Electric_Car_Footprints:ECE_Logo
- removed J3: Conn_01x04_Male, Connector_PinHeader_2.54mm:PinHeader_1x04_P2.54mm_Vertical
- removed J7: Conn_01x03_Male, Connector_PinHeader_2.54mm:PinHeader_1x03_P2.54mm_Horizontal
- removed R10, R11, R4, R5, R6, R7: 20k, Resistor_SMD:R_0805_2012Metric_Pad1.15x1.40mm_HandSolder
- removed R27: 61, Resistor_SMD:R_0805_2012Metric_Pad1.15x1.40mm_HandSolder
- removed R8, R9: 5k, Resistor_SMD:R_0805_2012Metric_Pad1.15x1.40mm_HandSolder
- removed SW2: SW_DIP_x04, Button_Switch_SMD:SW_DIP_SPSTx04_Slide_Omron_A6H-4101_W6.15mm_P1.27mm
- removed U2: MCP9808, Package_SO:MSOP-8_3x3mm_P0.65mm
- added F1: Fuse, Lafayette_Electric_Car_Footprints:fuse_holder_smd_littelfuse, F.Cu at (107.0, 111.3)
- added F2: Fuse, Lafayette_Electric_Car_Footprints:fuse_holder_smd_littelfuse, F.Cu at (174.5, 112.3)
- C1: value C -> 0.33uF
- C2: value C -> 0.1uF
- C7, C8, JP2, R1, R19, R2, R20, R22, R23, R3, TH1: moved to F.Cu
- H1, H2: footprint MountingHole:MountingHole_2.5mm_Pad -> Lafayette_Electric_Car_Footprints:SlottedHole
- J1: value Conn_01x04_Female -> Conn_01x04_Male; footprint Connector_PinHeader_2.54mm:PinHeader_1x04_P2.54mm_Horizontal -> Connector_PinHeader_2.54mm:PinHeader_1x04_P2.54mm_Vertical
- J2: value Conn_01x04_Male -> Conn_02x03_Odd_Even; footprint Connector_PinHeader_2.54mm:PinHeader_1x04_P2.54mm_Vertical -> Connector_IDC:IDC-Header_2x03_P2.54mm_Vertical
- SW1: value SW_DIP_x06 -> SW_DIP_x04; footprint Button_Switch_SMD:SW_DIP_SPSTx06_Slide_Omron_A6H-6101_W6.15mm_P1.27mm -> Button_Switch_SMD:SW_DIP_SPSTx04_Slide_Omron_A6H-4101_W6.15mm_P1.27mm
- U1: value ADC128D818 -> L7833CD-TR; footprint Package_SO:TSSOP-16_4.4x5mm_P0.65mm -> Package_SO:SO-8_3.9x4.9mm_P1.27mm
- moved J5 142.5 mm to (245.6, 49.7)
- moved J6 142.5 mm to (298.9, 49.0)
- moved JP2 46.1 mm to (166.6, 123.3), turned to 0 degrees
- moved JP1 43.9 mm to (165.3, 119.3), turned to 90 degrees
- moved C2 33.0 mm to (144.1, 90.8)
- moved C1 27.4 mm to (132.8, 90.9)
- moved D1 24.6 mm to (134.5, 96.2), turned to 180 degrees
- moved R13 23.6 mm to (134.4, 98.3), turned to 0 degrees
- moved R24 22.6 mm to (147.7, 116.7), turned to 180 degrees
- moved Q1 22.3 mm to (139.8, 96.4), turned to 0 degrees
- moved R12 20.8 mm to (139.8, 99.0), turned to 0 degrees
- moved J2 20.4 mm to (122.5, 89.2), turned to 0 degrees
- moved R18 20.0 mm to (143.7, 105.7), turned to 180 degrees
- moved R19 19.5 mm to (144.6, 112.9)
- moved C5 18.9 mm to (143.7, 103.6), turned to 0 degrees
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Connections:
- net /Indicator renamed /User_LED
- net Net-(JP1-Pad1) renamed /voltage_measurement/Prot_Cell+
- net Net-(R19-Pad1) renamed /Cell+(DIV)
- C1 pad 1: +3V3 -> /Seg+
- C1 pad 2: GND -> /Seg-
- C2 pad 2: GND -> /Seg-
- D1 pad 2: GND -> /Seg-
- H1 pad 1: /Cell+ -> Net-(F2-Pad2)
- H2 pad 1: /Cell- -> Net-(F1-Pad2)
- J2 pad 1: +3V3 -> /SCL
- J2 pad 2: /SDA -> /Seg+
- J2 pad 3: /SCL -> /SDA
- J2 pad 4: GND -> /Seg-
- J4 pad 1: /BalanceCurrent -> /Feedback
- J4 pad 2: /Feedback -> /BalanceCurrent
- J4 pad 3: /Balance_ctl -> /BalanceCurrent
- JP1 pad 2: Net-(JP1-Pad2) -> /Cell+
- JP2 pad 2: Net-(JP1-Pad2) -> /Cell+
- MCU1 pad 1: /Balance_ctl -> /BalanceCurrent
- MCU1 pad 16: Net-(MCU1-Pad16) -> /Address_0
- MCU1 pad 20: /Extra -> /Temperature
- MCU1 pad 3: /Temperature -> /Cell-(DIV)
- MCU1 pad 5: Net-(MCU1-Pad5) -> /Address_1
- MCU1 pad 6: Net-(MCU1-Pad6) -> /Address_2
- Q1 pad 2: GND -> /Seg-
- R1 pad 1: /Address_T0 -> /Address_2
- R12 pad 1: GND -> /Seg-
- R13 pad 1: +3V3 -> /Seg+
- R2 pad 2: /Address_T1 -> /Address_1
- R20 pad 1: Net-(R20-Pad1) -> /Cell-(DIV)
- R3 pad 2: /Address_T2 -> /Address_0
- SW1 pad 1: /Address_T0 -> /Address_2
- SW1 pad 2: /Address_T1 -> /Address_1
- SW1 pad 3: /Address_T2 -> /Address_0
- SW1 pad 4: /Address_G0 -> Net-(SW1-Pad4)
- SW1 pad 5: /Address_G1 -> /SafeGND
- SW1 pad 6: /Address_G2 -> /SafeGND
- U1 pad 1: Net-(U1-Pad1) -> +3V3
- U1 pad 2: /SDA -> /Seg-
- U1 pad 3: /SCL -> /Seg-
- U1 pad 4: /SafeGND -> Net-(U1-Pad4)
- U1 pad 5: +3V3 -> Net-(U1-Pad5)
- U1 pad 6: Net-(R7-Pad1) -> /Seg-
- U1 pad 7: /Address_A0 -> /Seg-
- U1 pad 8: /Address_A1 -> /Seg+
- U3 pad 8: Net-(R20-Pad1) -> /Cell-(DIV)
- U3 pad 9: Net-(R20-Pad1) -> /Cell-(DIV)
Routing:
- net +3V3: track 219.8 -> 24.8 mm, vias 10 -> 0
- net /Cell-: track 94.4 -> 0.00 mm, vias 5 -> 0
- net GND: track 90.0 -> 0.00 mm, vias 5 -> 0
- net /SafeGND: track 92.6 -> 21.8 mm, vias 16 -> 9
- net /SCL: track 107.2 -> 42.4 mm, vias 4 -> 1
- net /SDA: track 100.4 -> 42.8 mm, vias 4 -> 1
- net /Cell-(DIV): track 0.00 -> 36.1 mm
- net /Extra: track 34.1 -> 0.00 mm, vias 2 -> 0
- net /Address_T2: track 31.8 -> 0.00 mm, vias 2 -> 0
- net /Address_T1: track 29.2 -> 0.00 mm, vias 2 -> 0
- net /Address_T0: track 28.2 -> 0.00 mm, vias 2 -> 0
- net /Balance_ctl: track 26.2 -> 0.00 mm
- net /Cell+: track 25.8 -> 1.06 mm, vias 5 -> 0
- net /Address_A0: track 17.8 -> 0.00 mm
- net /Address_A1: track 17.5 -> 0.00 mm
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- removed copper zone on B.Cu, net /Cell+
- removed copper zone on F.Cu, net /Cell+
- removed copper zone on B.Cu, net /Cell-
- removed copper zone on B.Cu, net /SafeGND
Other:
- board text removed: "Address Select"
- board text removed: "Programming Interface"
- board text removed: "WARNING DO NOT LICK!"

Commit message: KiCad says there are no more traces to route, but my heart says otherwise
Parts:
- moved J6 203.7 mm to (108.4, 121.0), turned to 90 degrees
- moved J5 103.6 mm to (171.1, 121.7), turned to 90 degrees
- moved F1 68.8 mm to (175.7, 115.0), turned to 0 degrees
- moved F2 68.1 mm to (106.4, 114.1), turned to 180 degrees
- moved JP1 12.8 mm to (152.6, 120.5)
- moved JP2 12.8 mm to (153.9, 124.5)
- moved R3 8.75 mm to (159.3, 114.5), turned to 90 degrees
- moved R1 8.40 mm to (155.4, 114.5), turned to 270 degrees
- moved R2 7.64 mm to (157.4, 114.5), turned to 90 degrees
- moved R16 6.79 mm to (126.9, 121.0), turned to 180 degrees
- moved SW1 5.90 mm to (158.1, 107.9), turned to 90 degrees
- moved J4 5.67 mm to (173.3, 91.5)
- moved J1 4.54 mm to (147.3, 86.0)
- moved TH1 3.82 mm to (120.2, 104.5), turned to 90 degrees
- moved R14 2.88 mm to (117.0, 104.6), turned to 90 degrees
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Connections:
- F1 pad 1: /Cell- -> /Cell+
- F2 pad 1: /Cell+ -> /Cell-
- J4 pad 2: /BalanceCurrent -> /Balance_ctl
- MCU1 pad 1: /BalanceCurrent -> /Balance_ctl
- R1 pad 1: /Address_2 -> /Address_0
- R1 pad 2: +3V3 -> /SafeGND
- R2 pad 1: +3V3 -> /SafeGND
- R3 pad 1: +3V3 -> /SafeGND
- R3 pad 2: /Address_0 -> /Address_2
- SW1 pad 1: /Address_2 -> /Address_0
- SW1 pad 3: /Address_0 -> /Address_2
- SW1 pad 5: /SafeGND -> +3V3
- SW1 pad 6: /SafeGND -> +3V3
- SW1 pad 7: /SafeGND -> +3V3
- SW1 pad 8: /SafeGND -> +3V3
Routing:
- net +3V3: track 24.8 -> 110.6 mm, vias 0 -> 6
- net /Cell+: track 1.06 -> 66.3 mm
- net /Cell-: track 0.00 -> 41.2 mm
- net /Seg-: track 16.0 -> 50.5 mm
- net /SafeGND: track 21.8 -> 51.7 mm, vias 9 -> 17
- net /Address_0: track 4.47 -> 28.6 mm, vias 1 -> 2
- net /Address_2: track 2.84 -> 24.0 mm
- net /Seg+: track 3.37 -> 24.4 mm, vias 0 -> 3
- net /Address_1: track 2.56 -> 23.3 mm
- net /Balance_ctl: track 0.00 -> 20.2 mm, vias 0 -> 2
- net /BalanceCurrent: track 41.1 -> 24.6 mm
- net Net-(F1-Pad2): track 0.00 -> 10.8 mm
- net Net-(F2-Pad2): track 1.88 -> 12.4 mm
- net /SCL: track 42.4 -> 34.2 mm
- net /SDA: track 42.8 -> 39.6 mm
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- added copper zone on B.Cu, net /SafeGND

Commit message: approved?
Parts:
- H1, H2: footprint Lafayette_Electric_Car_Footprints:SlottedHole -> Lafayette_Electric_Car_Footprints:CellMan_Mount_InHouse
- moved H2 0.17 mm to (175.2, 105.4), turned to 180 degrees
- moved H1 0.11 mm to (106.5, 105.5), turned to 180 degrees
Connections:
- net Net-(F1-Pad2) renamed /Cell+(RAW)
- net Net-(F2-Pad2) renamed /Cell-(RAW)
Routing:
- net /Cell-(RAW): track 12.4 -> 5.91 mm
- added copper zone on B.Cu, net (none)
- added copper zone on F.Cu, net /Cell-(RAW)
Changed lines of the file:
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@@
     (thickness 1.6)
     (drawings 18)
-    (tracks 353)
+    (tracks 349)
     (zones 0)
     (modules 43)
@@
     (trace_clearance 0.254)
     (zone_clearance 0.508)
-    (zone_45_only no)
+    (zone_45_only yes)
     (trace_min 0)
     (via_size 0.8)
@@
   (net 39 "Net-(J2-Pad5)")
   (net 40 /voltage_measurement/Prot_Cell+)
-  (net 41 "Net-(F1-Pad2)")
-  (net 42 "Net-(F2-Pad2)")
+  (net 41 "/Cell+(RAW)")
+  (net 42 "/Cell-(RAW)")
   (net_class Default "This is the default net class."
     (clearance 0.254)
@@
     (add_net /Cell+)
     (add_net "/Cell+(DIV)")
+    (add_net "/Cell+(RAW)")
     (add_net /Cell-)
     (add_net "/Cell-(DIV)")
+    (add_net "/Cell-(RAW)")
     (add_net /CellVoltage)
     (add_net /Extra)
@@
     (add_net "Net-(D2-Pad1)")
     (add_net "Net-(D3-Pad2)")
-    (add_net "Net-(F1-Pad2)")
-    (add_net "Net-(F2-Pad2)")
     (add_net "Net-(J2-Pad5)")
     (add_net "Net-(J2-Pad6)")
@@
     (add_net "Net-(U1-Pad5)")
     (add_net "Net-(U3-Pad6)")
+  )
+  (module Lafayette_Electric_Car_Footprints:CellMan_Mount_InHouse (layer F.Cu)
+    (at 175.18 105.4 180)
+    (fp_text reference H2 (at 0 -8.21) (layer F.SilkS)
+      (effects (font (size 1 1) (thickness 0.15)))
+    )
+    (fp_text value MountingHole_Pad (at 0 -9.21) (layer F.Fab)
+      (effects (font (size 1 1) (thickness 0.15)))
+    )
+    (fp_text user "Drill Here" (at 6.4 -3.48 270) (layer F.SilkS)
+      (effects (font (size 1 1) (thickness 0.15)))
+    )
+    (pad 3 smd oval (at 0 0 270) (size 3.81 5.715) (layers F.SilkS))
+    (pad 2 smd oval (at 0 0 270) (size 6.35 8.255) (layers F.Mask))
+    (pad 1 smd oval (at 0 0 270) (size 2.794 4.6736) (layers F.Cu F.Paste)
+      (net 41 "/Cell+(RAW)"))
+  )
+  (module Lafayette_Electric_Car_Footprints:CellMan_Mount_InHouse (layer F.Cu)
+    (at 106.51 105.46 180)
+    (fp_text reference H1 (at 0 -8.21) (layer F.SilkS)
+      (effects (font (size 1 1) (thickness 0.15)))
+    )
+    (fp_text value MountingHole_Pad (at 0 -9.21) (layer F.Fab)
+      (effects (font (size 1 1) (thickness 0.15)))
+    )
+    (pad 3 smd oval (at 0 0 270) (size 3.81 5.715) (layers F.SilkS))
+    (pad 2 smd oval (at 0 0 270) (size 6.35 8.255) (layers F.Mask))
+    (pad 1 smd oval (at 0 0 270) (size 2.794 4.6736) (layers F.Cu F.Paste)
+      (net 42 "/Cell-(RAW)"))
   )
   (module Connector_IDC:IDC-Header_2x03_P2.54mm_Vertical (layer F.Cu)
@@
     )
   )
-  (module Lafayette_Electric_Car_Footprints:SlottedHole (layer F.Cu)
-    (at 175.01 105.38)
-    (fp_text reference H2 (at -3.32 -3.09) (layer F.SilkS)
-      (effects (font (size 1 1) (thickness 0.15)))
-    )
-    (fp_text value MountingHole_Pad (at 3.73 -3.14) (layer F.Fab)
-      (effects (font (size 1 1) (thickness 0.15)))
-    )
-    (pad 1 thru_hole oval (at 0 0 90) (size 4.5 6.5) (drill oval 2.5 4.5) (layers *.Cu *.Mask)
-      (net 41 "Net-(F1-Pad2)"))
-  )
-  (module Lafayette_Electric_Car_Footprints:SlottedHole (layer F.Cu)
-    (at 106.43 105.38)
-    (fp_text reference H1 (at -3.32 -3.09) (layer F.SilkS)
-      (effects (font (size 1 1) (thickness 0.15)))
-    )
-    (fp_text value MountingHole_Pad (at 3.73 -3.14) (layer F.Fab)
-      (effects (font (size 1 1) (thickness 0.15)))
-    )
-    (pad 1 thru_hole oval (at 0 0 90) (size 4.5 6.5) (drill oval 2.5 4.5) (layers *.Cu *.Mask)
-      (net 42 "Net-(F2-Pad2)"))
-  )
   (module Lafayette_Electric_Car_Footprints:fuse_holder_smd_littelfuse (layer F.Cu)
     (at 106.36 114.14 180)
@@
     )
     (pad 2 smd rect (at 3.16 -0.42 180) (size 4.24 3.81) (layers F.Cu F.Paste F.Mask)
-      (net 42 "Net-(F2-Pad2)"))
+      (net 42 "/Cell-(RAW)"))
     (pad 1 smd rect (at -3.23 -0.42 180) (size 4.24 3.81) (layers F.Cu F.Paste F.Mask)
       (net 7 /Cell-))
@@
     )
     (pad 2 smd rect (at 3.16 -0.42) (size 4.24 3.81) (layers F.Cu F.Paste F.Mask)
-      (net 41 "Net-(F1-Pad2)"))
+      (net 41 "/Cell+(RAW)"))
     (pad 1 smd rect (at -3.23 -0.42) (size 4.24 3.81) (layers F.Cu F.Paste F.Mask)
       (net 6 /Cell+))
@@
     (effects (font (size 4 4) (thickness 0.5)) (justify left))
   )
-  (gr_text + (at 83.59 106.44 90) (layer F.SilkS)
+  (gr_text + (at 102.69 104.75 90) (layer F.SilkS)
     (effects (font (size 4 4) (thickness 0.5)) (justify left))
   )
@@
   (segment (start 117.0825 103.7025) (end 116.97 103.59) (width 0.25) (layer F.Cu) (net 10))
   (segment (start 120.25 103.7025) (end 117.0825 103.7025) (width 0.25) (layer F.Cu) (net 10))
-  (segment (start 106.43 105.38) (end 106.65 105.38) (width 1.5) (layer F.Cu) (net 42))
-  (segment (start 106.43 105.38) (end 107.442 106.392) (width 1.5) (layer F.Cu) (net 42))
-  (segment (start 106.202 105.38) (end 106.43 105.38) (width 1.5) (layer B.Cu) (net 42))
   (segment (start 155.34 120.76) (end 155.115 120.535) (width 0.25) (layer F.Cu) (net 6))
   (segment (start 155.45 115.505) (end 157.4 115.505) (width 0.25) (layer F.Cu) (net 1))
@@
   (segment (start 175.01 105.38) (end 175.01 105.39) (width 1.5) (layer F.Cu) (net 41))
   (segment (start 175.01 105.39) (end 178.83 109.21) (width 1.5) (layer F.Cu) (net 41))
-  (segment (start 103.2 108.61) (end 106.43 105.38) (width 1.5) (layer F.Cu) (net 42))
   (segment (start 103.2 114.52) (end 103.2 108.61) (width 1.5) (layer F.Cu) (net 42))
   (zone (net 0) (net_name "") (layer F.Cu) (hatch edge 0.508)
@@
       )
     )
+  )
+  (zone (net 1) (net_name /SafeGND) (layer B.Cu) (hatch edge 0.508)
+    (connect_pads (clearance 0.508))
+    (min_thickness 0.254)
+    (fill yes (arc_segments 32) (thermal_gap 0.508) (thermal_bridge_width 0.508))
+    (polygon
+      (pts
+        (xy 132.99 118.58) (xy 147.34 118.58) (xy 147.34 122.59) (xy 132.99 122.59)
+      )
+    )
+  )
+  (zone (net 42) (net_name "/Cell-(RAW)") (layer F.Cu) (hatch edge 0.508)
+    (connect_pads no (clearance 0.508))
+    (min_thickness 0.254)
+    (fill yes (arc_segments 32) (thermal_gap 0.508) (thermal_bridge_width 0.508))
+    (polygon
+      (pts
+        (xy 98.903469 100.25503) (xy 111.883469 98.95503) (xy 113.593469 111.93503) (xy 97.913469 110.19503)
+      )
+    )
+  )
+  (zone (net 0) (net_name "") (layer B.Cu) (hatch edge 0.508)
+    (connect_pads (clearance 0.508))
+    (min_thickness 0.254)
+    (fill yes (arc_segments 32) (thermal_gap 0.508) (thermal_bridge_width 0.508))
+    (polygon
+      (pts
+        (xy 97.6 91.946628) (xy 107.39 91.946628) (xy 107.39 99.776628) (xy 97.6 99.776628)
+      )
+    )

Commit message: some cleaning up
Parts:
- removed C5: 1uF, Capacitor_SMD:C_0805_2012Metric_Pad1.15x1.40mm_HandSolder
- removed D1: LED, LED_SMD:LED_0805_2012Metric
- removed H1, H2: MountingHole_Pad, Lafayette_Electric_Car_Footprints:CellMan_Mount_InHouse
- removed R12: 0, Resistor_SMD:R_0805_2012Metric_Pad1.15x1.40mm_HandSolder
- removed R13: R, Resistor_SMD:R_0805_2012Metric_Pad1.15x1.40mm_HandSolder
- added BT1: Battery_Cell, Lafayette_Electric_Car_Footprints:CELL60AH, F.Cu at (175.7, 105.0)
- added C3: 1uF, Capacitor_SMD:C_0805_2012Metric_Pad1.15x1.40mm_HandSolder, F.Cu at (142.4, 99.6)
- added G***: LOGO, Lafayette_Electric_Car_Footprints:ECE_Logo, B.Cu at (109.0, 91.4)
- added G***: LOGO, Lafayette_Electric_Car_Footprints:paw_solder_mask, F.Cu at (112.8, 86.4)
- added Q2: BSS138W, Package_TO_SOT_SMD:SOT-323_SC-70_Handsoldering, F.Cu at (129.8, 111.6)
- moved Q1 17.4 mm to (148.2, 111.6), turned to 270 degrees
- moved C7 7.72 mm to (141.1, 112.9), turned to 0 degrees
- moved R24 7.61 mm to (140.2, 118.0), turned to 90 degrees
- moved C8 7.36 mm to (136.9, 112.9), turned to 180 degrees
- moved R23 5.72 mm to (136.9, 115.0), turned to 180 degrees
- moved R22 5.36 mm to (141.1, 115.0), turned to 0 degrees
- moved R19 4.17 mm to (143.3, 109.0)
- moved U3 4.17 mm to (139.0, 107.2)
- moved R17 4.17 mm to (143.3, 105.1)
- moved R18 4.17 mm to (142.4, 101.7)
- moved R20 4.17 mm to (134.8, 107.1)
- moved R25 4.07 mm to (137.8, 118.0), turned to 90 degrees
- moved TH1 3.56 mm to (116.7, 105.1), turned to 270 degrees
- moved R14 3.06 mm to (120.0, 104.9), turned to 270 degrees
- moved D3 2.51 mm to (147.3, 94.4), turned to 90 degrees
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Connections:
- C6 pad 1: /SafeGND -> /Seg-
- C7 pad 2: /SafeGND -> /Seg-
- C8 pad 2: /SafeGND -> /Seg-
- C9 pad 2: /SafeGND -> /Seg-
- D3 pad 1: /SafeGND -> /Seg-
- J1 pad 3: /SafeGND -> /Seg-
- J2 pad 1: /SCL -> /Seg+
- J2 pad 2: /Seg+ -> /Seg-
- J2 pad 3: /SDA -> /SCL
- J2 pad 4: /Seg- -> /SDA
- J2 pad 5: Net-(J2-Pad5) -> /Seg-
- J2 pad 6: Net-(J2-Pad6) -> /Seg+
- J4 pad 4: /Extra -> (no net)
- J4 pad 6: /SafeGND -> /Seg-
- MCU1 pad 10: Net-(MCU1-Pad10) -> (no net)
- MCU1 pad 13: Net-(MCU1-Pad13) -> (no net)
- MCU1 pad 15: Net-(MCU1-Pad15) -> (no net)
- MCU1 pad 2: /CellVoltage -> /Cell-(DIV)
- MCU1 pad 3: /Cell-(DIV) -> /CellVoltage
- MCU1 pad 7: /SafeGND -> /Seg-
- Q1 pad 3: /SafeGND -> Net-(Q1-Pad3)
- R1 pad 2: /SafeGND -> /Seg-
- R14 pad 1: /SafeGND -> /Seg-
- R18 pad 1: /SafeGND -> /Seg-
- R2 pad 1: /SafeGND -> /Seg-
- R22 pad 2: /SafeGND -> Net-(Q1-Pad3)
- R23 pad 2: /SafeGND -> Net-(Q2-Pad3)
- R3 pad 1: /SafeGND -> /Seg-
- SW1 pad 4: Net-(SW1-Pad4) -> (no net)
- U1 pad 4: Net-(U1-Pad4) -> (no net)
- U1 pad 5: Net-(U1-Pad5) -> (no net)
- U3 pad 11: /SafeGND -> /Seg-
Routing:
- net /SafeGND: track 51.7 -> 0.00 mm, vias 17 -> 0
- net +3V3: track 110.6 -> 136.8 mm, vias 6 -> 5
- net /SDA: track 39.6 -> 29.0 mm
- net /Cell-: track 41.2 -> 50.8 mm
- net /Seg-: track 50.5 -> 59.1 mm, vias 0 -> 17
- net Net-(Q1-Pad3): track 0.00 -> 7.52 mm
- net Net-(Q2-Pad3): track 0.00 -> 7.43 mm
- net Net-(C7-Pad1): track 14.4 -> 7.06 mm
- net /voltage_measurement/Prot_Cell+: track 10.4 -> 17.4 mm
- net /SCL: track 34.2 -> 40.8 mm, vias 1 -> 3
- net Net-(C8-Pad1): track 13.5 -> 7.04 mm
- net /Cell-(RAW): track 5.91 -> 11.5 mm, vias 0 -> 4
- net /Cell-(DIV): track 36.6 -> 31.6 mm, vias 0 -> 2
- net Net-(D1-Pad1): track 2.06 -> 0.00 mm
- net /Address_0: track 28.6 -> 30.6 mm
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- added copper zone on B.Cu, net /Cell+(RAW)
- added copper zone on F.Cu, net /Cell+(RAW)
- added copper zone on B.Cu, net /Cell-(RAW)
- added copper zone on B.Cu, net /Seg-
- removed copper zone on B.Cu, net (none)
- removed copper zone on F.Cu, net /Cell-
- removed copper zone on B.Cu, net /SafeGND
Other:
- board size 100 x 45 mm -> 99.1 x 45.7 mm
- board text added: "CellMan v1.4"
- board text added: "Connor Winiarczyk '20"
- board text added: "Reverse Cell Polarity"
- board text removed: "CellMan v1.0"
- board text removed: "Connor Winiarczyk"
- board text removed: "Plugged In Backwards!"
